File: 4272ShaftEncoder_R2/4272ShaftEncoder.kicad_pcb (KiCad board)
At the start: 2 copper layers, 15.9 x 23.3 mm, 13 parts, among them J1 Strain3, U1 AS5600-ASOM

Commit message: Add pre-season archive
Parts:
- added TP1: TestPoint, TestPoint:TestPoint_THTPad_1.0x1.0mm_Drill0.5mm, F.Cu at (141.2, 77.8)
- added TP2: TestPoint, TestPoint:TestPoint_THTPad_1.0x1.0mm_Drill0.5mm, F.Cu at (141.2, 79.9)
- added TP3: TestPoint, TestPoint:TestPoint_THTPad_1.0x1.0mm_Drill0.5mm, F.Cu at (143.7, 82.4)
Connections:
- net Net-(R1-Pad2) renamed /DIR
- net Net-(R6-Pad1) renamed /SDA
- net Net-(R7-Pad1) renamed /SCL
- U1 pad 5: unconnected-(U1-Pad5) -> /PGO
Routing:
- net /SDA: track 8.38 -> 13.0 mm
- net /SCL: track 12.3 -> 16.4 mm
- net /PGO: track 0.00 -> 3.05 mm
- net +3.3V: track 38.8 -> 38.1 mm
- net GND: track 7.05 -> 7.21 mm, vias 15 -> 14
Other:
- board text added: "PGO"
- board text added: "REV3"
- board text added: "SCL"
- board text added: "SDA"
- board text removed: "REV2"
