File: 4272ShaftEncoder_R2/4272ShaftEncoder.kicad_sch (KiCad schematic)
At the start: 12 parts, among them J1 Strain3, U1 AS5600-ASOM

Commit message: Add pre-season archive
Parts:
- added TP1, TP2, TP3: TestPoint, TestPoint:TestPoint_THTPad_1.0x1.0mm_Drill0.5mm, symbol Connector:TestPoint
Connections:
- net DIR: now reaches R1.2, R2.1, U1.8 (DIR)
- net PGO: now reaches U1.5 (PGO)
- net PGO: now also TP3.1
- net SDA: now reaches R6.1, U1.6 (SDA)
- net SDA: now also TP2.1
- net SCL: now reaches R7.1, U1.7 (SCL)
- net SCL: now also TP1.1
Changed lines of the file:
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@@
   (junction (at 217.805 106.68) (diameter 0) (color 0 0 0 0)
   )
+  (junction (at 184.15 109.22) (diameter 0) (color 0 0 0 0)
+  )
   (junction (at 139.7 109.22) (diameter 0) (color 0 0 0 0)
   )
@@
   (junction (at 127 111.76) (diameter 0) (color 0 0 0 0)
   )
+  (junction (at 193.675 111.76) (diameter 0) (color 0 0 0 0)
+  )
   (wire (pts (xy 139.7 109.22) (xy 124.46 109.22))
     (stroke (width 0) (type default) (color 0 0 0 0))
@@
     (stroke (width 0) (type default) (color 0 0 0 0))
   )
+  (wire (pts (xy 172.72 114.3) (xy 184.15 114.3))
+    (stroke (width 0) (type default) (color 0 0 0 0))
+  )
   (wire (pts (xy 217.805 106.68) (xy 217.805 107.95))
     (stroke (width 0) (type default) (color 0 0 0 0))
@@
   (wire (pts (xy 92.71 116.84) (xy 127 116.84))
     (stroke (width 0) (type default) (color 0 0 0 0))
+  )
+  (label "PGO" (at 174.625 114.3 0)
+    (effects (font (size 1.27 1.27)) (justify left bottom))
   )
   (label "CW" (at 224.155 111.76 0)
     (effects (font (size 1.27 1.27)) (justify left bottom))
   )
+  (label "SDA" (at 174.625 111.76 0)
+    (effects (font (size 1.27 1.27)) (justify left bottom))
+  )
+  (label "SCL" (at 174.625 109.22 0)
+    (effects (font (size 1.27 1.27)) (justify left bottom))
+  )
   (label "OUT" (at 130.81 111.76 0)
     (effects (font (size 1.27 1.27)) (justify left bottom))
   )
   (label "CCW" (at 222.885 99.695 0)
+    (effects (font (size 1.27 1.27)) (justify left bottom))
+  )
+  (label "DIR" (at 174.625 106.68 0)
     (effects (font (size 1.27 1.27)) (justify left bottom))
   )
@@
     )
     (property "Datasheet" "" (id 3) (at 217.805 115.57 0)
+      (effects (font (size 1.27 1.27)) hide)
+    )
+    (pin "1")
+  )
+  (symbol (lib_id "Connector:TestPoint") (at 193.675 111.76 270) (unit 1)
+    (in_bom yes) (on_board yes) (fields_autoplaced)
+    (property "Reference" "TP2" (id 0) (at 199.39 111.7599 90)
+      (effects (font (size 1.27 1.27)) (justify left))
+    )
+    (property "Value" "TestPoint" (id 1) (at 199.39 113.0299 90)
+      (effects (font (size 1.27 1.27)) (justify left) hide)
+    )
+    (property "Footprint" "TestPoint:TestPoint_THTPad_1.0x1.0mm_Drill0.5mm" (id 2) (at 193.675 116.84 0)
+      (effects (font (size 1.27 1.27)) hide)
+    )
+    (property "Datasheet" "~" (id 3) (at 193.675 116.84 0)
       (effects (font (size 1.27 1.27)) hide)
     )
@@
     (pin "3")
   )
+  (symbol (lib_id "Connector:TestPoint") (at 184.15 114.3 270) (unit 1)
+    (in_bom yes) (on_board yes) (fields_autoplaced)
+    (property "Reference" "TP3" (id 0) (at 189.865 114.2999 90)
+      (effects (font (size 1.27 1.27)) (justify left))
+    )
+    (property "Value" "TestPoint" (id 1) (at 189.865 115.5699 90)
+      (effects (font (size 1.27 1.27)) (justify left) hide)
+    )
+    (property "Footprint" "TestPoint:TestPoint_THTPad_1.0x1.0mm_Drill0.5mm" (id 2) (at 184.15 119.38 0)
+      (effects (font (size 1.27 1.27)) hide)
+    )
+    (property "Datasheet" "~" (id 3) (at 184.15 119.38 0)
+      (effects (font (size 1.27 1.27)) hide)
+    )
+    (pin "1")
+  )
   (symbol (lib_id "power:+3.3V") (at 184.15 90.805 0) (unit 1)
     (in_bom yes) (on_board yes) (fields_autoplaced)
@@
     (pin "1")
     (pin "2")
+  )
+  (symbol (lib_id "Connector:TestPoint") (at 184.15 109.22 270) (unit 1)
+    (in_bom yes) (on_board yes)
+    (property "Reference" "TP1" (id 0) (at 188.595 107.95 90)
+      (effects (font (size 1.27 1.27)) (justify left))
+    )
+    (property "Value" "TestPoint" (id 1) (at 182.245 111.125 90)
+      (effects (font (size 1.27 1.27)) (justify left) hide)
+    )
+    (property "Footprint" "TestPoint:TestPoint_THTPad_1.0x1.0mm_Drill0.5mm" (id 2) (at 184.15 114.3 0)
+      (effects (font (size 1.27 1.27)) hide)
+    )
+    (property "Datasheet" "~" (id 3) (at 184.15 114.3 0)
+      (effects (font (size 1.27 1.27)) hide)
+    )
+    (pin "1")
   )
   (symbol (lib_id "pspice:CAP") (at 127 128.27 0) (unit 1)
@@
       (reference "R7") (unit 1) (value "100K") (footprint "Resistor_SMD:R_0603_1608Metric_Pad0.98x0.95mm_HandSolder")
     )
+    (path "/a40372be-6e8c-4435-ab0e-f4e6ea139c6f"
+      (reference "TP1") (unit 1) (value "TestPoint") (footprint "TestPoint:TestPoint_THTPad_1.0x1.0mm_Drill0.5mm")
+    )
+    (path "/50d5a694-93b6-4e62-89cd-cfffb4d91efa"
+      (reference "TP2") (unit 1) (value "TestPoint") (footprint "TestPoint:TestPoint_THTPad_1.0x1.0mm_Drill0.5mm")
+    )
+    (path "/8c89ae4f-ba52-4bcd-ac0f-21b5cd04ab76"
+      (reference "TP3") (unit 1) (value "TestPoint") (footprint "TestPoint:TestPoint_THTPad_1.0x1.0mm_Drill0.5mm")
+    )
     (path "/21f97db3-0506-4b51-9248-711f81c6fe38"
